File: project/4GBMemoryUSB.kicad_pcb (KiCad board)
At the start: 2 copper layers, 20 x 36.2 mm, 12 parts, among them J1 USB_A, J2 Conn_01x06_Socket, U1 LD1117S33TR_SOT223

Commit message: Update with photos + fix LED VCC
Connections:
- R1 pad 1: Net-(J1-VBUS) -> Net-(J2-Pin_1)
Routing:
- net Net-(J2-Pin_1): track 28.0 -> 35.4 mm
- net Net-(J1-VBUS): track 16.3 -> 14.9 mm
Other:
- rule pad_to_mask_clearance: 0.0508 -> 0
Changed lines of the file:
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@@
 			(dielectric_constraints no)
 		)
-		(pad_to_mask_clearance 0.0508)
+		(pad_to_mask_clearance 0)
 		(allow_soldermask_bridges_in_footprints no)
 		(tenting
@@
 		(capping no)
 		(filling no)
-		(zone_defaults)
 		(pcbplotparams
 			(layerselection 0x00000000_00000000_55555555_5755f5ff)
@@
 		)
 		(property "Value" "10uF"
-			(at 0 1.5 0)
+			(at 0 1.2 0)
 			(layer "F.Fab")
 			(effects
@@
 			(layers "F.Cu" "F.Mask" "F.Paste")
 			(roundrect_rratio 0.25)
-			(net "Net-(J1-VBUS)")
+			(net "Net-(J2-Pin_1)")
 			(pintype "passive")
 		)
@@
 	)
 	(segment
+		(start 105.3375 82)
+		(end 104.6 82)
+		(width 0.2)
+		(layer "F.Cu")
+		(net "Net-(J2-Pin_1)")
+	)
+	(segment
+		(start 104.4 84.8)
+		(end 105 85.4)
+		(width 0.2)
+		(layer "F.Cu")
+		(net "Net-(J2-Pin_1)")
+	)
+	(segment
 		(start 105.5 98.850002)
 		(end 105.5 95.15)
@@
 	)
 	(segment
+		(start 105.55 85.4)
+		(end 107.25 87.1)
+		(width 0.2)
+		(layer "F.Cu")
+		(net "Net-(J2-Pin_1)")
+	)
+	(segment
 		(start 105.5 95.15)
 		(end 107.25 93.4)
@@
 	)
 	(segment
+		(start 105 85.4)
+		(end 105.55 85.4)
+		(width 0.2)
+		(layer "F.Cu")
+		(net "Net-(J2-Pin_1)")
+	)
+	(segment
 		(start 109.75 97)
 		(end 111.3625 97)
@@
 	)
 	(segment
+		(start 104.4 82.2)
+		(end 104.4 84.8)
+		(width 0.2)
+		(layer "F.Cu")
+		(net "Net-(J2-Pin_1)")
+	)
+	(segment
 		(start 103.75 93)
 		(end 106.85 93)
@@
 	)
 	(segment
+		(start 104.6 82)
+		(end 104.4 82.2)
+		(width 0.2)
+		(layer "F.Cu")
+		(net "Net-(J2-Pin_1)")
+	)
+	(segment
 		(start 104 80)
 		(end 104 79.25)
@@
 		(width 0.2)
 		(layer "F.Cu")
-		(net "Net-(J1-VBUS)")
-	)
-	(segment
-		(start 105.3375 82)
-		(end 104 82)
-		(width 0.2)
-		(layer "F.Cu")
